File: SemuBot_WheelBase/Wheelbase/Wheelbase.kicad_sch (KiCad schematic)
At the start: 19 parts, among them IC1 NCP164CSN330T1G, J1 10155435-00011LF, J2 ftsh-105-01-l-dv-k, U1 STM32F303RET6, Y1 WE-SPXO_CFPS-39

Commit message: Snapshot
Parts:
- added D2: DEBUG_LED, LED_SMD:LED_0603_1608Metric_Pad1.05x0.95mm_HandSolder, symbol Device:LED
- added D3: PRTR5V0U2X, Package_TO_SOT_SMD:SOT-143, symbol Power_Protection:PRTR5V0U2X
- added J3: TB003-500-P02BE, TB003-500-P02BE:CUI_TB003-500-P02BE, symbol TB003-500-P02BE:TB003-500-P02BE
- added J4, J5, J6: B5B-XH-A_LF__SN_, B5B-XH-A_LF__SN_:JST_B5B-XH-A_LF__SN_, symbol B5B-XH-A_LF__SN_:B5B-XH-A_LF__SN_
- added J7, J8, J9: 1984620, 1984620:PHOENIX_1984620, symbol 1984620:1984620
- added R6: 3.3K, Resistor_SMD:R_0603_1608Metric_Pad0.98x0.95mm_HandSolder, symbol Device:R
- C1, C10, C11, C12, C13, C14, C15, C2, C3: footprint (none) -> Capacitor_SMD:C_0603_1608Metric_Pad1.08x0.95mm_HandSolder
- D1: footprint (none) -> LED_SMD:LED_0201_0603Metric_Pad0.64x0.40mm_HandSolder
- J1: footprint 10155435-00011LF:AMPHENOL_10155435-00011LF -> library:AMPHENOL_10155435-00011LF
- J2: footprint FTSH-105-XX-X-DV:SAMTEC_FTSH-105-XX-X-DV -> library:SAMTEC_FTSH-105-XX-X-DV
- R1, R2, R3, R5: footprint (none) -> Resistor_SMD:R_0603_1608Metric_Pad0.98x0.95mm_HandSolder
Connections:
- net +5V: now also D3.4 (VCC), J4.1, J5.1, J6.1
- net D+: now also D3.3 (I/O2)
- net D-: now also D3.2 (I/O1)
- net Motor_1/HAL_1: now also J4.4
- net Motor_1/HAL_2: now also J4.3
- net Motor_1/HAL_3: now also J4.2
- net Motor_1/MA: now also J9.1
- net Motor_1/MB: now also J9.2
- net Motor_1/MC: now also J9.3
- net GND: now also U1.60 (BOOT0), D3.1 (GND), J4.5, J5.5, J6.5, R6.2
- net MOTOR2_PWM: now reaches U1.22 (PA6)
- net nBRAKE: now reaches U1.33 (PB12)
- net ENABLE: now reaches U1.36 (PB15)
- net at U1.37 (PC6): now also D2.2 (A)
- net CS_ENC_3: now reaches U1.38 (PC7)
- net CS_ENC_2: now reaches U1.39 (PC8)
- net CS_ENC_1: now reaches U1.40 (PC9)
- net MOTOR3_DIR: now reaches U1.41 (PA8)
- net MOTOR2_DIR: now reaches U1.42 (PA9)
- net MOTOR1_DIR: now reaches U1.43 (PA10)
- net MOTOR3_PWM: now reaches U1.58 (PB6)
- net MOTOR1_PWM: now reaches U1.8 (PC0)
- new net: D2.1 (K), R6.1
- new net +24V: J3.2 (24V+)
- new net Motor_2/HAL_1: J5.4
- new net Motor_2/HAL_2: J5.3
- new net Motor_2/HAL_3: J5.2
- new net Motor_2/MA: J8.1
- new net Motor_2/MB: J8.2
- new net Motor_2/MC: J8.3
- new net Motor_3/HAL_1: J6.4
- new net Motor_3/HAL_2: J6.3
- new net Motor_3/HAL_3: J6.2
- new net Motor_3/MA: J7.1
- new net Motor_3/MB: J7.2
- new net Motor_3/MC: J7.3
- new net PGND: J3.1 (GND)
- no-connect marks 2 -> 38
Other:
- sheet Driver renamed Motor_1
- added sheet Motor_2 (Driver.kicad_sch)
- added sheet Motor_3 (Driver.kicad_sch)
- sheet Motor_1 ports: added ENABLE; removed none
- note added: "24V input"
- note added: "USB ESD Protection"
- moved on the sheet: J1, J2, R1, R2

Commit message: Snapshot
Parts:
- added J10, J11, J12: B5B-XH-A_LF__SN_, B5B-XH-A_LF__SN_:JST_B5B-XH-A_LF__SN_, symbol B5B-XH-A_LF__SN_:B5B-XH-A_LF__SN_
Connections:
- net +24V: now also J3.1 (24V); no longer J3.2 (24V+)
- net +5V: now also J10.1, J11.1, J12.1
- net CS_ENC_1: now also J10.4
- net CS_ENC_2: now also J11.4
- net CS_ENC_3: now also J12.4
- net GND: now also J10.5, J11.5, J12.5
- net MOTOR1_DIR: now also U1.29 (PB10); no longer U1.43 (PA10)
- net MOTOR2_DIR: now also U1.28 (PB2); no longer U1.42 (PA9)
- net MOTOR3_DIR: now also U1.27 (PB1); no longer U1.41 (PA8)
- net Motor_1/MA: now also J9.3; no longer J9.1
- net Motor_1/MC: now also J9.1; no longer J9.3
- net Motor_2/MA: now also J8.3; no longer J8.1
- net Motor_2/MC: now also J8.1; no longer J8.3
- net Motor_3/MA: now also J7.3; no longer J7.1
- net Motor_3/MC: now also J7.1; no longer J7.3
- net PGND: now also J3.2 (PGND); no longer J3.1 (GND)
- net at D2.2 (A): now also U1.2 (PC13); no longer U1.37 (PC6)
- net SPI_CLK: now reaches U1.34 (PB13)
- net SPI_CLK: now also J10.3, J11.3, J12.3
- net SPI_DATA: now reaches U1.35 (PB14)
- net SPI_DATA: now also J10.2, J11.2, J12.2
- no-connect marks 38 -> 27
Other:
- moved on the sheet: D2, J3, R6

Commit message: Snapshot
Connections:
- net +3.3V: now also U1.1 (VBAT), U1.13 (VDDA), U1.19 (VDD), U1.32 (VDD), U1.48 (VDD), U1.64 (VDD)
- net CS_ENC_1: now also U1.29 (PB10); no longer U1.40 (PC9)
- net CS_ENC_2: now also U1.30 (PB11); no longer U1.39 (PC8)
- net CS_ENC_3: now also U1.33 (PB12); no longer U1.38 (PC7)
- net ENABLE: now also U1.27 (PB1); no longer U1.36 (PB15)
- net GND: no longer U1.1 (VBAT), U1.13 (VDDA), U1.19 (VDD), U1.32 (VDD), U1.48 (VDD), U1.64 (VDD)
- net MOTOR1_DIR: now also U1.28 (PB2); no longer U1.29 (PB10)
- net MOTOR2_DIR: now also U1.20 (PA4); no longer U1.28 (PB2)
- net MOTOR3_DIR: now also U1.25 (PC5); no longer U1.27 (PB1)
- net nBRAKE: now also U1.26 (PB0); no longer U1.33 (PB12)
- no-connect marks 27 -> 32
Other:
- moved on the sheet: C12, C13, C14, C15

Commit message: Snapshot
Parts:
- added H1: MH1, MountingHole:MountingHole_2.2mm_M2_Pad_Via, symbol Mechanical:MountingHole_Pad
- added H2: MH2, MountingHole:MountingHole_2.2mm_M2_Pad_Via, symbol Mechanical:MountingHole_Pad
- added H3: MH3, MountingHole:MountingHole_2.2mm_M2_Pad_Via, symbol Mechanical:MountingHole_Pad
- added H4: MH4, MountingHole:MountingHole_2.2mm_M2_Pad_Via, symbol Mechanical:MountingHole_Pad
Connections:
- net PGND is gone; now on net GND: J3.2 (PGND)
- net CS_ENC_1: now also U1.36 (PB15); no longer U1.29 (PB10)
- net CS_ENC_2: now also U1.17 (PA3); no longer U1.30 (PB11)
- net CS_ENC_3: now also U1.37 (PC6); no longer U1.33 (PB12)
- net ENABLE: now also U1.33 (PB12); no longer U1.27 (PB1)
- net GND: now also H1.1, H2.1, H3.1, H4.1
- net MOTOR1_DIR: now also U1.30 (PB11); no longer U1.28 (PB2)
- net MOTOR2_DIR: now also U1.21 (PA5); no longer U1.20 (PA4)
- net MOTOR3_DIR: now also U1.28 (PB2); no longer U1.25 (PC5)
- net Motor_1/HAL_1: now also J4.2; no longer J4.4
- net Motor_1/HAL_3: now also J4.4; no longer J4.2
- net Motor_2/HAL_1: now also J5.2; no longer J5.4
- net Motor_2/HAL_3: now also J5.4; no longer J5.2
- net Motor_3/HAL_1: now also J6.2; no longer J6.4
- net Motor_3/HAL_3: now also J6.4; no longer J6.2
- net nBRAKE: now also U1.29 (PB10); no longer U1.26 (PB0)
- no-connect marks 32 -> 36

Commit message: Revision time
Other:
- moved on the sheet: D2, R6
Changed lines of the file:
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@@
 	(wire
 		(pts
-			(xy 69.85 115.57) (xy 71.12 115.57)
+			(xy 92.71 133.35) (xy 92.71 132.08)
 		)
 		(stroke
@@
 	(wire
 		(pts
-			(xy 87.63 115.57) (xy 100.33 115.57)
+			(xy 92.71 115.57) (xy 100.33 115.57)
 		)
 		(stroke
@@
 	(wire
 		(pts
-			(xy 78.74 115.57) (xy 80.01 115.57)
+			(xy 92.71 124.46) (xy 92.71 123.19)
 		)
 		(stroke
@@
 	(symbol
 		(lib_id "power:GND")
-		(at 69.85 115.57 0)
+		(at 92.71 133.35 90)
 		(unit 1)
 		(exclude_from_sim no)
@@
 		(fields_autoplaced yes)
 		(property "Reference" "#PWR011"
-			(at 69.85 121.92 0)
+			(at 99.06 133.35 0)
 			(effects
 				(font
@@
 		)
 		(property "Value" "GND"
-			(at 69.85 120.65 0)
+			(at 97.79 133.35 0)
 			(effects
 				(font
@@
 		)
 		(property "Footprint" ""
-			(at 69.85 115.57 0)
+			(at 92.71 133.35 0)
 			(effects
 				(font
@@
 		)
 		(property "Datasheet" ""
-			(at 69.85 115.57 0)
+			(at 92.71 133.35 0)
 			(effects
 				(font
@@
 		)
 		(property "Description" "Power symbol creates a global label with name \"GND\" , ground"
-			(at 69.85 115.57 0)
+			(at 92.71 133.35 0)
 			(effects
 				(font
@@
 	(symbol
 		(lib_id "Device:LED")
-		(at 83.82 115.57 0)
+		(at 92.71 119.38 90)
 		(unit 1)
 		(exclude_from_sim no)
@@
 		(fields_autoplaced yes)
 		(property "Reference" "D2"
-			(at 82.2325 109.22 0)
+			(at 86.36 120.9675 0)
 			(effects
 				(font
@@
 		)
 		(property "Value" "DEBUG_LED"
-			(at 82.2325 111.76 0)
+			(at 88.9 120.9675 0)
 			(effects
 				(font
@@
 		)
 		(property "Footprint" "LED_SMD:LED_0603_1608Metric_Pad1.05x0.95mm_HandSolder"
-			(at 83.82 115.57 0)
+			(at 92.71 119.38 0)
 			(effects
 				(font
@@
 		)
 		(property "Datasheet" "~"
-			(at 83.82 115.57 0)
+			(at 92.71 119.38 0)
 			(effects
 				(font
@@
 		)
 		(property "Description" "Light emitting diode"
-			(at 83.82 115.57 0)
+			(at 92.71 119.38 0)
 			(effects
 				(font
@@
 	(symbol
 		(lib_id "Device:R")
-		(at 74.93 115.57 270)
+		(at 92.71 128.27 0)
 		(unit 1)
 		(exclude_from_sim no)
@@
 		(dnp no)
 		(property "Reference" "R6"
-			(at 74.676 119.126 90)
+			(at 96.266 128.524 90)
 			(effects
 				(font
@@
 		)
 		(property "Value" "3.3K"
-			(at 74.168 117.602 90)
+			(at 94.742 129.032 90)
 			(effects
 				(font
@@
 		)
 		(property "Footprint" "Resistor_SMD:R_0603_1608Metric_Pad0.98x0.95mm_HandSolder"
-			(at 74.93 113.792 90)
+			(at 90.932 128.27 90)
 			(effects
 				(font
@@
 		)
 		(property "Datasheet" "~"
-			(at 74.93 115.57 0)
+			(at 92.71 128.27 0)
 			(effects
 				(font
@@
 		)
 		(property "Description" "Resistor"
-			(at 74.93 115.57 0)
+			(at 92.71 128.27 0)
 			(effects
 				(font

Commit message: Final version atm
Parts:
- added D7: +24V, LED_SMD:LED_0603_1608Metric_Pad1.05x0.95mm_HandSolder, symbol Device:LED
- added D8: +3.3V, LED_SMD:LED_0603_1608Metric_Pad1.05x0.95mm_HandSolder, symbol Device:LED
- added R18: 1.2K, Resistor_SMD:R_0603_1608Metric_Pad0.98x0.95mm_HandSolder, symbol Device:R
- added R19: 3.3K, Resistor_SMD:R_0603_1608Metric_Pad0.98x0.95mm_HandSolder, symbol Device:R
- D1: footprint LED_SMD:LED_0201_0603Metric_Pad0.64x0.40mm_HandSolder -> LED_SMD:LED_0603_1608Metric_Pad1.05x0.95mm_HandSolder
Connections:
- net +24V: now also D7.2 (A)
- net +3.3V: now also D8.2 (A)
- net GND: now also R18.2, R19.2
- new net: D8.1 (K), R19.1
- new net: D7.1 (K), R18.1
