File: SemuBot_WheelBase/Wheelbase/Wheelbase.kicad_pcb (KiCad board)
At the start: 2 copper layers, 60 x 60 mm, 71 parts, among them IC1 NCP164CSN330T1G, J1 10155435-00011LF, J2 ftsh-105-01-l-dv-k, J3 TB003-500-P02BE, J4 B5B-XH-A_LF__SN_, J5 B5B-XH-A_LF__SN_, J6 B5B-XH-A_LF__SN_, J7 1984620, J8 1984620, J9 1984620, Q1 DI025N06PT-AQ, Q10 DI025N06PT-AQ, Q11 DI025N06PT-AQ, Q12 DI025N06PT-AQ, Q13 DI025N06PT-AQ, Q14 DI025N06PT-AQ, Q15 DI025N06PT-AQ, Q16 DI025N06PT-AQ, Q17 DI025N06PT-AQ, Q18 DI025N06PT-AQ, Q2 DI025N06PT-AQ, Q3 DI025N06PT-AQ, Q4 DI025N06PT-AQ, Q5 DI025N06PT-AQ, Q6 DI025N06PT-AQ, Q7 DI025N06PT-AQ, Q8 DI025N06PT-AQ, Q9 DI025N06PT-AQ, U1 STM32F303RET6, U2 DRV8353FSRTAR, U3 DRV8353FSRTAR, U4 DRV8353FSRTAR, Y1 WE-SPXO_CFPS-39

Commit message: Snapshot
Parts:
- added J10: B5B-XH-A_LF__SN_, B5B-XH-A_LF__SN_:JST_B5B-XH-A_LF__SN_, F.Cu at (192.9, 74.5)
- added J11: B5B-XH-A_LF__SN_, B5B-XH-A_LF__SN_:JST_B5B-XH-A_LF__SN_, F.Cu at (183.3, 74.5)
- added J12: B5B-XH-A_LF__SN_, B5B-XH-A_LF__SN_:JST_B5B-XH-A_LF__SN_, F.Cu at (173.8, 74.5)
- added R10: 1k, Resistor_SMD:R_0603_1608Metric_Pad0.98x0.95mm_HandSolder, F.Cu at (131.7, 85.5)
- added R11: 1k, Resistor_SMD:R_0603_1608Metric_Pad0.98x0.95mm_HandSolder, F.Cu at (142.6, 111.0)
- added R12: 1k, Resistor_SMD:R_0603_1608Metric_Pad0.98x0.95mm_HandSolder, F.Cu at (175.9, 88.1)
- added R13: 1k, Resistor_SMD:R_0603_1608Metric_Pad0.98x0.95mm_HandSolder, F.Cu at (135.3, 102.0)
- added R14: 1k, Resistor_SMD:R_0603_1608Metric_Pad0.98x0.95mm_HandSolder, F.Cu at (162.1, 110.0)
- added R15: 1k, Resistor_SMD:R_0603_1608Metric_Pad0.98x0.95mm_HandSolder, F.Cu at (173.6, 101.6)
- added R16: 1k, Resistor_SMD:R_0603_1608Metric_Pad0.98x0.95mm_HandSolder, F.Cu at (131.0, 92.2)
- added R17: 1k, Resistor_SMD:R_0603_1608Metric_Pad0.98x0.95mm_HandSolder, F.Cu at (148.2, 113.3)
- added R9: 1k, Resistor_SMD:R_0603_1608Metric_Pad0.98x0.95mm_HandSolder, F.Cu at (173.0, 105.1)
- moved J3 73.6 mm to (177.4, 117.7), turned to 180 degrees
- moved J7 63.4 mm to (158.4, 123.2), turned to 180 degrees
- moved Q18 56.1 mm to (162.4, 118.2), turned to -90 degrees
- moved Q17 50.8 mm to (158.3, 118.2), turned to 90 degrees
- moved R8 47.4 mm to (158.5, 108.4)
- moved Q15 45.3 mm to (154.2, 118.2), turned to 90 degrees
- moved C24 44.8 mm to (158.4, 110.5)
- moved J5 43.5 mm to (144.3, 94.5)
- moved J6 42.2 mm to (152.1, 94.4)
- moved Q16 41.9 mm to (150.2, 118.2), turned to -90 degrees
- moved C4 38.7 mm to (164.5, 101.8), turned to -90 degrees
- moved C5 38.4 mm to (166.3, 101.8), turned to -90 degrees
- moved C26 38.3 mm to (149.2, 104.3)
- moved C25 38.0 mm to (149.3, 102.8), turned to 180 degrees
- moved Q13 37.9 mm to (145.9, 118.2), turned to 90 degrees
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Connections:
- J3 pad 1: PGND -> +24V
- J3 pad 2: +24V -> PGND
- J7 pad 1: /Motor_3/SHA -> /Motor_3/SHC
- J7 pad 3: /Motor_3/SHC -> /Motor_3/SHA
- J8 pad 1: /Motor_2/SHA -> /Motor_2/SHC
- J8 pad 3: /Motor_2/SHC -> /Motor_2/SHA
- J9 pad 1: /Motor_1/SHA -> /Motor_1/SHC
- J9 pad 3: /Motor_1/SHC -> /Motor_1/SHA
- U1 pad 2: unconnected-(U1-PC13-Pad2) -> Net-(D2-A)
- U1 pad 27: unconnected-(U1-PB1-Pad27) -> /MOTOR3_DIR
- U1 pad 28: unconnected-(U1-PB2-Pad28) -> /MOTOR2_DIR
- U1 pad 29: unconnected-(U1-PB10-Pad29) -> /MOTOR1_DIR
- U1 pad 34: unconnected-(U1-PB13-Pad34) -> /SPI_CLK
- U1 pad 35: unconnected-(U1-PB14-Pad35) -> /SPI_DATA
- U1 pad 37: Net-(D2-A) -> unconnected-(U1-PC6-Pad37)
- U1 pad 41: /MOTOR3_DIR -> unconnected-(U1-PA8-Pad41)
- U1 pad 42: /MOTOR2_DIR -> unconnected-(U1-PA9-Pad42)
- U1 pad 43: /MOTOR1_DIR -> unconnected-(U1-PA10-Pad43)
- U2 pad 10: unconnected-(U2-SNA-Pad10) -> PGND
- U2 pad 11: unconnected-(U2-SNB-Pad11) -> PGND
- U2 pad 20: unconnected-(U2-SNC-Pad20) -> PGND
- U3 pad 10: unconnected-(U3-SNA-Pad10) -> PGND
- U3 pad 11: unconnected-(U3-SNB-Pad11) -> PGND
- U3 pad 20: unconnected-(U3-SNC-Pad20) -> PGND
- U4 pad 10: unconnected-(U4-SNA-Pad10) -> PGND
- U4 pad 11: unconnected-(U4-SNB-Pad11) -> PGND
- U4 pad 20: unconnected-(U4-SNC-Pad20) -> PGND
Routing:
- net +5V: track 83.3 -> 218.7 mm
- net /MOTOR3_PWM: track 0.00 -> 78.3 mm, vias 0 -> 2
- net /ENABLE: track 0.00 -> 73.3 mm, vias 0 -> 6
- net /nBRAKE: track 21.9 -> 79.8 mm, vias 2 -> 8
- net /MOTOR2_DIR: track 0.00 -> 48.4 mm, vias 0 -> 2
- net /MOTOR3_DIR: track 0.00 -> 47.1 mm, vias 0 -> 2
- net /MOTOR2_PWM: track 0.00 -> 46.8 mm, vias 0 -> 2
- net /CS_ENC_2: track 0.00 -> 45.9 mm
- net /CS_ENC_1: track 0.00 -> 36.1 mm, vias 0 -> 2
- net /MOTOR1_PWM: track 67.1 -> 35.3 mm, vias 2 -> 4
- net /SPI_CLK: track 0.00 -> 28.8 mm
- net +24V: track 0.14 -> 28.7 mm
- net /SPI_DATA: track 0.00 -> 27.2 mm
- net /Motor_3/SHA: track 0.00 -> 19.1 mm, vias 0 -> 2
- net /Motor_3/SHC: track 0.00 -> 19.0 mm, vias 0 -> 2
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- added copper zone on F.Cu, net +24V
- added copper zone on F.Cu, net /Motor_1/SHA
- added copper zone on F.Cu, net /Motor_1/SHB
- added copper zone on F.Cu, net /Motor_1/SHC
- added copper zone on F.Cu, net /Motor_2/SHA
- added copper zone on F.Cu, net /Motor_2/SHB
- added copper zone on F.Cu, net /Motor_2/SHC
- added copper zone on F.Cu, net /Motor_3/SHA
- added copper zone on F.Cu, net /Motor_3/SHB
- added copper zone on F.Cu, net /Motor_3/SHC
Other:
- board size 60 x 60 mm -> 84 x 81.5 mm
- rule pad_to_mask_clearance: 0 -> 0.05

Commit message: Snapshot
Parts:
- moved J1 74.1 mm to (114.5, 73.7), turned to -90 degrees
- moved C2 66.3 mm to (120.9, 80.3), turned to 180 degrees
- moved D1 61.3 mm to (123.6, 80.3), turned to 180 degrees
- moved C1 61.1 mm to (122.7, 77.9), turned to -90 degrees
- moved R2 59.4 mm to (122.4, 74.9), turned to 180 degrees
- moved R1 58.7 mm to (122.1, 70.8), turned to -90 degrees
- moved R3 55.0 mm to (127.0, 80.0), turned to 180 degrees
- moved IC1 53.5 mm to (126.4, 77.1), turned to 0 degrees
- moved D3 51.6 mm to (126.0, 73.2), turned to -90 degrees
- moved J3 47.9 mm to (129.5, 116.2)
- moved C12 29.2 mm to (145.4, 83.2), turned to 180 degrees
- moved C13 28.4 mm to (145.4, 81.7), turned to 180 degrees
- moved C14 27.8 mm to (145.4, 80.0), turned to 180 degrees
- moved C15 27.3 mm to (145.4, 78.5), turned to 180 degrees
- moved J2 18.0 mm to (165.9, 71.1)
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Connections:
- U1 pad 1: GND -> +3.3V
- U1 pad 13: GND -> +3.3V
- U1 pad 19: GND -> +3.3V
- U1 pad 20: unconnected-(U1-PA4-Pad20) -> /MOTOR2_DIR
- U1 pad 25: unconnected-(U1-PC5-Pad25) -> /MOTOR3_DIR
- U1 pad 26: unconnected-(U1-PB0-Pad26) -> /nBRAKE
- U1 pad 27: /MOTOR3_DIR -> /ENABLE
- U1 pad 28: /MOTOR2_DIR -> /MOTOR1_DIR
- U1 pad 29: /MOTOR1_DIR -> /CS_ENC_1
- U1 pad 30: unconnected-(U1-PB11-Pad30) -> /CS_ENC_2
- U1 pad 32: GND -> +3.3V
- U1 pad 33: /nBRAKE -> /CS_ENC_3
- U1 pad 36: /ENABLE -> unconnected-(U1-PB15-Pad36)
- U1 pad 38: /CS_ENC_3 -> unconnected-(U1-PC7-Pad38)
- U1 pad 39: /CS_ENC_2 -> unconnected-(U1-PC8-Pad39)
- U1 pad 40: /CS_ENC_1 -> unconnected-(U1-PC9-Pad40)
- U1 pad 48: GND -> +3.3V
- U1 pad 64: GND -> +3.3V
Routing:
- net +3.3V: track 23.6 -> 91.5 mm, vias 0 -> 8
- net /MOTOR3_PWM: track 78.3 -> 41.1 mm, vias 2 -> 4
- net +5V: track 218.7 -> 255.0 mm, vias 0 -> 3
- net /D+: track 16.6 -> 44.7 mm, vias 0 -> 2
- net /D-: track 17.9 -> 45.7 mm, vias 0 -> 2
- net GND: track 6.32 -> 32.3 mm, vias 6 -> 45
- net /MOTOR2_DIR: track 48.4 -> 23.2 mm
- net /MOTOR2_PWM: track 46.8 -> 27.7 mm
- net PGND: track 0.00 -> 16.7 mm, vias 0 -> 22
- net /MOTOR3_DIR: track 47.1 -> 30.8 mm
- net /nBRAKE: track 79.8 -> 64.2 mm, vias 8 -> 5
- net /CS_ENC_2: track 45.9 -> 30.9 mm
- net /Motor_3/SPA: track 6.73 -> 18.8 mm
- net /Motor_2/SPC: track 7.09 -> 17.8 mm, vias 0 -> 2
- net /ENABLE: track 73.3 -> 63.0 mm, vias 6 -> 5
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- added copper zone on B.Cu, net GND
- added copper zone on F.Cu, net GND
- added copper zone on B.Cu, net PGND
- added copper zone on F.Cu, net PGND
Other:
- board size 84 x 81.5 mm -> 84 x 65 mm

Commit message: Snapshot
Parts:
- moved R17 0.25 mm to (148.2, 113.1)
Routing:
- net /Motor_3/SPA: track 18.8 -> 21.1 mm, vias 2 -> 4

Commit message: Snapshot
Parts:
- added D4: LED, LED_SMD:LED_0603_1608Metric_Pad1.05x0.95mm_HandSolder, F.Cu at (169.0, 90.5)
- added D5: LED, LED_SMD:LED_0603_1608Metric_Pad1.05x0.95mm_HandSolder, F.Cu at (138.1, 99.2)
- added D6: LED, LED_SMD:LED_0603_1608Metric_Pad1.05x0.95mm_HandSolder, F.Cu at (157.7, 107.0)
- added H1: MH1, MountingHole:MountingHole_2.2mm_M2_Pad_Via, F.Cu at (117.0, 127.0)
- added H2: MH2, MountingHole:MountingHole_2.2mm_M2_Pad_Via, F.Cu at (193.0, 127.0)
- added H3: MH3, MountingHole:MountingHole_2.2mm_M2_Pad_Via, F.Cu at (193.0, 70.0)
- added H4: MH4, MountingHole:MountingHole_2.2mm_M2_Pad_Via, F.Cu at (130.8, 69.0)
- moved J11 75.3 mm to (116.7, 109.5), turned to -90 degrees
- moved J12 51.8 mm to (167.6, 126.0), turned to 0 degrees
- moved J10 39.9 mm to (188.6, 114.1)
- moved J5 14.1 mm to (135.9, 83.1), turned to 0 degrees
- moved J4 12.1 mm to (167.2, 84.7), turned to 0 degrees
- moved J3 9.45 mm to (130.0, 125.7)
- moved J6 4.42 mm to (153.4, 98.6), turned to 0 degrees
- moved R8 3.31 mm to (158.6, 104.5)
- moved R7 2.75 mm to (141.4, 99.3)
- moved R13 1.84 mm to (134.6, 100.3)
- moved R4 1.68 mm to (169.0, 88.8), turned to 0 degrees
- moved C12 0.86 mm to (146.1, 82.8)
- moved C13 0.86 mm to (146.1, 81.2)
- moved C14 0.86 mm to (146.1, 79.5)
- moved C15 0.86 mm to (146.1, 78.0)
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Connections:
- J3 pad 2: PGND -> GND
- J4 pad 2: /Motor_1/HAL_3 -> /Motor_1/HAL_1
- J4 pad 4: /Motor_1/HAL_1 -> /Motor_1/HAL_3
- J5 pad 2: /Motor_2/HAL_3 -> /Motor_2/HAL_1
- J5 pad 4: /Motor_2/HAL_1 -> /Motor_2/HAL_3
- J6 pad 2: /Motor_3/HAL_3 -> /Motor_3/HAL_1
- J6 pad 4: /Motor_3/HAL_1 -> /Motor_3/HAL_3
- R10 pad 1: PGND -> GND
- R11 pad 1: PGND -> GND
- R12 pad 1: PGND -> GND
- R13 pad 1: PGND -> GND
- R14 pad 1: PGND -> GND
- R15 pad 1: PGND -> GND
- R16 pad 1: PGND -> GND
- R17 pad 1: PGND -> GND
- R4 pad 1: Net-(U2-~{FAULT}) -> Net-(D4-A)
- R7 pad 1: Net-(U3-~{FAULT}) -> Net-(D5-A)
- R8 pad 1: Net-(U4-~{FAULT}) -> Net-(D6-A)
- R9 pad 1: PGND -> GND
- U1 pad 17: unconnected-(U1-PA3-Pad17) -> /CS_ENC_2
- U1 pad 20: /MOTOR2_DIR -> unconnected-(U1-PA4-Pad20)
- U1 pad 21: unconnected-(U1-PA5-Pad21) -> /MOTOR2_DIR
- U1 pad 25: /MOTOR3_DIR -> unconnected-(U1-PC5-Pad25)
- U1 pad 26: /nBRAKE -> unconnected-(U1-PB0-Pad26)
- U1 pad 27: /ENABLE -> unconnected-(U1-PB1-Pad27)
- U1 pad 28: /MOTOR1_DIR -> /MOTOR3_DIR
- U1 pad 29: /CS_ENC_1 -> /nBRAKE
- U1 pad 30: /CS_ENC_2 -> /MOTOR1_DIR
- U1 pad 33: /CS_ENC_3 -> /ENABLE
- U1 pad 36: unconnected-(U1-PB15-Pad36) -> /CS_ENC_1
- U1 pad 37: unconnected-(U1-PC6-Pad37) -> /CS_ENC_3
- U2 pad 10: PGND -> GND
- U2 pad 11: PGND -> GND
- U2 pad 20: PGND -> GND
- U2 pad 25: PGND -> GND
- U2 pad 26: Net-(U2-~{FAULT}) -> Net-(D4-K)
- U2 pad 39: PGND -> GND
- U3 pad 10: PGND -> GND
- U3 pad 11: PGND -> GND
- U3 pad 20: PGND -> GND
- U3 pad 25: PGND -> GND
- U3 pad 26: Net-(U3-~{FAULT}) -> Net-(D5-K)
- U3 pad 39: PGND -> GND
- U4 pad 10: PGND -> GND
- U4 pad 11: PGND -> GND
- U4 pad 20: PGND -> GND
- U4 pad 25: PGND -> GND
- U4 pad 26: Net-(U4-~{FAULT}) -> Net-(D6-K)
- U4 pad 39: PGND -> GND
Routing:
- net /SPI_CLK: track 34.6 -> 157.9 mm, vias 0 -> 2
- net /SPI_DATA: track 35.4 -> 154.5 mm, vias 0 -> 2
- net +5V: track 255.0 -> 347.4 mm, vias 3 -> 1
- net /CS_ENC_3: track 14.5 -> 102.6 mm, vias 0 -> 1
- net /CS_ENC_2: track 30.9 -> 63.8 mm
- net /CS_ENC_1: track 40.4 -> 67.2 mm, vias 0 -> 2
- net GND: track 32.3 -> 54.6 mm, vias 45 -> 166
- net /Motor_2/HAL_2: track 6.10 -> 27.3 mm, vias 0 -> 2
- net /Motor_2/HAL_3: track 8.24 -> 28.5 mm, vias 0 -> 2
- net /Motor_2/HAL_1: track 5.93 -> 25.7 mm, vias 0 -> 2
- net PGND: track 16.7 -> 0.00 mm, vias 22 -> 0
- net /nBRAKE: track 64.2 -> 72.4 mm, vias 5 -> 10
- net /Motor_3/HAL_3: track 15.6 -> 7.79 mm
- net /Motor_3/HAL_2: track 13.1 -> 6.74 mm
- net /ENABLE: track 63.0 -> 69.1 mm, vias 5 -> 6
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- removed copper zone on B.Cu, net PGND
- removed copper zone on F.Cu, net PGND
Other:
- board text added: "+24V"
- board text added: "DEBUG"
- board text added: "GND"
- board text added: "MOTOR 1"
- board text added: "MOTOR 2"
- board text added: "MOTOR 3"
- board text added: "MOTOR2"
- board text added: "POWER"

Commit message: Revision time
Parts:
- moved R10 1.50 mm to (131.4, 86.9)
- moved R3 0.78 mm to (126.2, 79.9)
- moved C21 0.73 mm to (131.5, 89.6)
- moved J5 0.33 mm to (135.9, 82.8)
Connections:
- H1 pad 1: (no net) -> GND
Routing:
- net /Motor_1/SPC: track 3.70 -> 9.50 mm
- net /Motor_2/SPA: track 18.5 -> 14.9 mm
- net /D-: track 42.4 -> 44.7 mm
- net /Motor_2/GLA: track 16.5 -> 17.7 mm
- net GND: track 54.6 -> 55.4 mm, vias 166 -> 171
- net Net-(D1-K): track 2.17 -> 1.44 mm
- net +5V: track 347.4 -> 348.0 mm
- net Net-(J1-CC1): track 2.59 -> 3.13 mm

Commit message: Final version atm
Parts:
- added D7: +24V, LED_SMD:LED_0603_1608Metric_Pad1.05x0.95mm_HandSolder, F.Cu at (136.6, 105.2)
- added D8: +3.3V, LED_SMD:LED_0603_1608Metric_Pad1.05x0.95mm_HandSolder, F.Cu at (131.2, 76.6)
- added R18: 1.2K, Resistor_SMD:R_0603_1608Metric_Pad0.98x0.95mm_HandSolder, F.Cu at (139.9, 105.2)
- added R19: 3.3K, Resistor_SMD:R_0603_1608Metric_Pad0.98x0.95mm_HandSolder, F.Cu at (134.7, 76.7)
- D1: footprint LED_SMD:LED_0201_0603Metric_Pad0.64x0.40mm_HandSolder -> LED_SMD:LED_0603_1608Metric_Pad1.05x0.95mm_HandSolder
- moved R3 0.95 mm to (127.2, 79.9), turned to -90 degrees
- moved C2 0.78 mm to (120.3, 80.8)
- moved D1 0.58 mm to (123.7, 80.9)
Routing:
- net +3.3V: track 88.5 -> 91.2 mm
- net Net-(D8-K): track 0.00 -> 1.77 mm
- net Net-(D7-K): track 0.00 -> 1.52 mm
- net GND: track 55.4 -> 56.8 mm, vias 171 -> 178
- net Net-(D1-K): track 1.44 -> 2.61 mm
- net Net-(IC1-PG/ADJ): track 2.13 -> 1.17 mm

Commit message: Ver2
Parts:
- removed J2: ftsh-105-01-l-dv-k, library:SAMTEC_FTSH-105-XX-X-DV
- removed Y1: WE-SPXO_CFPS-39, WE-SPXO_CFPS-39:WE-SPXO_CFPS-39
- added J13: SSW-104-01-FM-D, SSW-104-01-FM-D:SAMTEC_SSW-104-01-FM-D, F.Cu at (165.0, 71.2)
- added Y2: X322516MLB4SI, X322516MLB4SI:OSC_X322516MLB4SI, F.Cu at (143.3, 73.0)
- R18: value 1.2K -> 3.3K
- moved C11 2.95 mm to (143.4, 70.5), turned to 180 degrees
- moved C10 1.70 mm to (141.7, 77.3)
- moved R5 1.70 mm to (141.7, 75.8)
Connections:
- C11 pad 1: GND -> /OSC_IN
- C11 pad 2: /OSC_IN -> GND
- R3 pad 2: Net-(D1-K) -> +3.3V
Routing:
- net /NRST: track 24.1 -> 33.4 mm
- net /SWCLK: track 7.73 -> 12.5 mm
- net GND: track 56.8 -> 52.5 mm, vias 178 -> 171
- net /OSC_IN: track 10.6 -> 6.53 mm
- net +3.3V: track 91.2 -> 87.1 mm, vias 5 -> 3
- net /OSC_OUT: track 10.3 -> 8.39 mm
- net /SWDIO: track 4.92 -> 6.03 mm
- net Net-(C10-Pad2): track 3.86 -> 4.45 mm

Commit message: Updating board
Parts:
- removed D1: LED, LED_SMD:LED_0603_1608Metric_Pad1.05x0.95mm_HandSolder
- added D9: +3.3V, LED_SMD:LED_0603_1608Metric_Pad1.05x0.95mm_HandSolder, F.Cu at (115.3, 80.0)
- added J2: MTSW-103-09-L-S-400, MTSW-103-09-L-S-400:SAMTEC_MTSW-103-09-L-S-400, F.Cu at (151.1, 85.2)
- added R20: 3.3K, Resistor_SMD:R_0603_1608Metric_Pad0.98x0.95mm_HandSolder, F.Cu at (115.3, 81.7)
- moved J13 5.14 mm to (170.1, 71.4)
- moved R3 0.59 mm to (127.0, 80.5)
- moved C19 0.10 mm to (139.5, 88.3)
- moved C20 0.10 mm to (139.5, 89.8)
Connections:
- U1 pad 15: unconnected-(U1-PA1-Pad15) -> /CS_ENC_2
- U1 pad 16: unconnected-(U1-PA2-Pad16) -> /USART2_TX
- U1 pad 17: /CS_ENC_2 -> /USART2_RX
Routing:
- net /USART2_TX: track 0.00 -> 7.23 mm
- net +3.3V: track 87.1 -> 92.9 mm
- net /USART2_RX: track 0.00 -> 5.23 mm
- net /NRST: track 33.4 -> 38.5 mm
- net /SWCLK: track 12.5 -> 17.5 mm
- net /SWDIO: track 6.03 -> 10.7 mm
- net /MOTOR2_PWM: track 23.1 -> 25.7 mm
- net Net-(D1-K): track 2.61 -> 0.00 mm
- net +5V: track 348.0 -> 350.4 mm
- net /CS_ENC_2: track 64.0 -> 66.1 mm
- net Net-(D9-K): track 0.00 -> 1.75 mm
- net /MOTOR2_DIR: track 23.7 -> 24.8 mm
- net GND: track 52.5 -> 53.5 mm, vias 171 -> 170
- net Net-(IC1-PG/ADJ): track 1.17 -> 1.81 mm
Other:
- board text added: "24V"
- board text added: "3.3V"
- board text added: "5V"
- board text added: "NRST"
- board text added: "RX"
- board text added: "SWCLK"
- board text added: "SWDI0"
- board text added: "TX"
