File: SemuBot_WheelBase/Wheelbase/Driver.kicad_sch (KiCad schematic)
At the start: 14 parts, among them Q1 DI025N06PT-AQ, Q2 DI025N06PT-AQ, Q3 DI025N06PT-AQ, Q4 DI025N06PT-AQ, Q5 DI025N06PT-AQ, Q6 DI025N06PT-AQ, U3 DRV8353FSRTAR

Commit message: Snapshot
Parts:
- C22: renamed from C4; footprint (none) -> Capacitor_SMD:C_0603_1608Metric_Pad1.08x0.95mm_HandSolder
- C23: renamed from C5; footprint (none) -> Capacitor_SMD:C_0603_1608Metric_Pad1.08x0.95mm_HandSolder
- C24: renamed from C6; footprint (none) -> Capacitor_SMD:C_0603_1608Metric_Pad1.08x0.95mm_HandSolder
- C25: renamed from C7; footprint (none) -> Capacitor_SMD:C_0603_1608Metric_Pad1.08x0.95mm_HandSolder
- C26: renamed from C8; footprint (none) -> Capacitor_SMD:C_0603_1608Metric_Pad1.08x0.95mm_HandSolder
- C27: renamed from C9; footprint (none) -> Capacitor_SMD:C_0603_1608Metric_Pad1.08x0.95mm_HandSolder
- R8: renamed from R4; footprint (none) -> Resistor_SMD:R_0603_1608Metric_Pad0.98x0.95mm_HandSolder
- U4: renamed from U3; footprint DRV8353HRTAT:QFN50P600X600X80-41N -> DRV8353HRTAT(1):QFN50P600X600X80-41N
- renumbered Q1 to Q13, Q2 to Q14, Q3 to Q15, Q4 to Q16, Q5 to Q17, Q6 to Q18
Connections:
- net GND: no longer U4.25 (AGND), U4.39 (GND)
- net ENABLE: now reaches U4.31 (ENABLE)
- new net PGND: U4.25 (AGND), U4.39 (GND)
- no-connect marks 3 -> 10
Other:
- moved on the sheet: C24, C25

Commit message: Snapshot
Parts:
- added R11, R14, R17: 1k, Resistor_SMD:R_0603_1608Metric_Pad0.98x0.95mm_HandSolder, symbol Device:R
Connections:
- net PGND: now also U4.10 (SNA), U4.11 (SNB), U4.20 (SNC), R11.1, R14.1, R17.1
- net SPA: now also R11.2
- net SPB: now also R17.2
- net SPC: now also R14.2
- no-connect marks 10 -> 7
Other:
- moved on the sheet: Q15, Q16

Commit message: Snapshot
Parts:
- added D4: LED, LED_SMD:LED_0603_1608Metric_Pad1.05x0.95mm_HandSolder, symbol Device:LED
Connections:
- net PGND is gone; now on net GND: R11.1, R14.1, R17.1, U4.10 (SNA), U4.11 (SNB), U4.20 (SNC), U4.25 (AGND), U4.39 (GND)
- net at U4.26 (~{FAULT}): now also D4.1 (K); no longer R8.1
- new net: D4.2 (A), R8.1
Other:
- moved on the sheet: R8

Commit message: Revision time
Parts:
- renumbered D4 to D6
Changed lines of the file:
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@@
 		(dnp no)
 		(fields_autoplaced yes)
-		(property "Reference" "D4"
+		(property "Reference" "D6"
 			(at 130.4925 62.23 0)
 			(effects
@@
 		(dnp no)
 		(fields_autoplaced yes)
-		(property "Reference" "#PWR069"
+		(property "Reference" "#PWR071"
 			(at 166.37 143.51 0)
 			(effects
@@
 		(dnp no)
 		(fields_autoplaced yes)
-		(property "Reference" "#PWR063"
+		(property "Reference" "#PWR065"
 			(at 210.82 71.12 0)
 			(effects
@@
 		(dnp no)
 		(fields_autoplaced yes)
-		(property "Reference" "#PWR036"
+		(property "Reference" "#PWR078"
 			(at 118.11 139.7 0)
 			(effects

Commit message: Ver2
Parts:
- renumbered C22 to C4, C23 to C5, C24 to C6, C25 to C7, C26 to C8, C27 to C9, D6 to D4, Q13 to Q1, Q14 to Q2, Q15 to Q3, Q16 to Q4, Q17 to Q5, Q18 to Q6, R14 to R12, R17 to R15, R8 to R4, R11 to R9, U4 to U2

Commit message: Snapshot
Parts:
- added R24, R27, R30, R33: 0, Resistor_SMD:R_0603_1608Metric_Pad0.98x0.95mm_HandSolder, symbol Device:R
Connections:
- net GND: now also R24.1, R27.1, R30.1, R33.1
- net MODE: now reaches U2.27 (MODE)
- net MODE: now also R30.2
- net IDRIVE: now reaches U2.28 (IDRIVE)
- net VDS: now reaches U2.29 (VDS)
- net VDS: now also R33.2
- net GAIN: now reaches U2.30 (GAIN)
- net GAIN: now also R24.2
- new net IDRIVe: R27.2
- no-connect marks 7 -> 3
